Commit message: cude

File: URDFrv4310V5/urdf/URDFrv4310V6.urdf (robot description, URDF)
Before this commit: robot URDFrv4310V5, 6 links, 5 joints
Joints:
- joint Joint_2: limit lower=-3 upper=3 effort=1 velocity=31 -> lower=-3 upper=3 effort=3 velocity=31
- joint Joint_3: limit lower=-1.8 upper=2.4 effort=1 velocity=31 -> lower=-1.8 upper=2.4 effort=35 velocity=31
- joint Joint_4: limit lower=-3 upper=0.9 effort=1 velocity=31 -> lower=-3 upper=0.9 effort=3 velocity=31
- joint Joint_5: limit lower=-4 upper=4 effort=1 velocity=31 -> lower=-4 upper=4 effort=3 velocity=31
- joint Joint_6: limit lower=-3.5 upper=0.9 effort=1 velocity=31 -> lower=-3.5 upper=0.9 effort=3 velocity=31
